File: Rev. 1/Eagle/C64_Kernal_Switch.brd (EAGLE design)
At the start: 20 x 101.2 mm, 33 parts, among them IC1 ATMEGA328P-AU, J1 M20-7862042C64KB, J2 WSL 6G, J3 n/a, Q1 BC846, X1 FOXSLF/160-20

Commit message: Rev. 1 Documentation released
The final documentation is released
Parts:
- R10: value 1k -> n/a
- R9: value 220R -> 330R
Changed lines of the file:
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@@
 <?xml version="1.0" encoding="utf-8"?>
 <!DOCTYPE eagle SYSTEM "eagle.dtd">
-<eagle version="9.2.2">
+<eagle version="9.5.2">
 <drawing>
 <settings>
@@
 <layer number="14" name="Route14" color="22" fill="1" visible="no" active="no"/>
 <layer number="15" name="Route15" color="23" fill="1" visible="no" active="no"/>
-<layer number="16" name="Bottom" color="1" fill="1" visible="no" active="yes"/>
-<layer number="17" name="Pads" color="2" fill="1" visible="no" active="yes"/>
-<layer number="18" name="Vias" color="2" fill="1" visible="no" active="yes"/>
+<layer number="16" name="Bottom" color="1" fill="1" visible="yes" active="yes"/>
+<layer number="17" name="Pads" color="2" fill="1" visible="yes" active="yes"/>
+<layer number="18" name="Vias" color="2" fill="1" visible="yes" active="yes"/>
 <layer number="19" name="Unrouted" color="6" fill="1" visible="yes" active="yes"/>
 <layer number="20" name="Dimension" color="24" fill="1" visible="yes" active="yes"/>
-<layer number="21" name="tPlace" color="7" fill="1" visible="yes" active="yes"/>
+<layer number="21" name="tPlace" color="7" fill="1" visible="no" active="yes"/>
 <layer number="22" name="bPlace" color="7" fill="1" visible="no" active="yes"/>
-<layer number="23" name="tOrigins" color="15" fill="1" visible="yes" active="yes"/>
+<layer number="23" name="tOrigins" color="15" fill="1" visible="no" active="yes"/>
 <layer number="24" name="bOrigins" color="15" fill="1" visible="no" active="yes"/>
 <layer number="25" name="tNames" color="7" fill="1" visible="no" active="yes"/>
 <layer number="26" name="bNames" color="7" fill="1" visible="no" active="yes"/>
-<layer number="27" name="tValues" color="7" fill="1" visible="yes" active="yes"/>
+<layer number="27" name="tValues" color="7" fill="1" visible="no" active="yes"/>
 <layer number="28" name="bValues" color="7" fill="1" visible="no" active="yes"/>
 <layer number="29" name="tStop" color="7" fill="3" visible="no" active="yes"/>
@@
 <layer number="49" name="Reference" color="7" fill="1" visible="no" active="yes"/>
 <layer number="50" name="dxf" color="7" fill="1" visible="no" active="no"/>
-<layer number="51" name="tDocu" color="7" fill="1" visible="yes" active="yes"/>
+<layer number="51" name="tDocu" color="7" fill="1" visible="no" active="yes"/>
 <layer number="52" name="bDocu" color="7" fill="1" visible="no" active="yes"/>
 <layer number="53" name="tGND_GNDA" color="7" fill="1" visible="no" active="no"/>
@@
 <attribute name="VALUE" x="7.096125" y="70.00875" size="1.016" layer="27" ratio="10" rot="R270"/>
 </element>
-<element name="R9" library="SMD" package="0805" value="220R" x="7.62" y="75.168125" smashed="yes" rot="R270">
+<element name="R9" library="SMD" package="0805" value="330R" x="7.62" y="75.168125" smashed="yes" rot="R270">
 <attribute name="NAME" x="6.842125" y="77.136625" size="1.016" layer="25" ratio="10"/>
 <attribute name="VALUE" x="7.1755" y="76.755625" size="1.016" layer="27" ratio="10" rot="R270"/>
 </element>
-<element name="R10" library="SMD" package="0805" value="1k" x="4.92125" y="3.254375" smashed="yes" rot="R270">
+<element name="R10" library="SMD" package="0805" value="n/a" x="4.92125" y="3.254375" smashed="yes" rot="R270">
 <attribute name="NAME" x="3.90525" y="1.2065" size="1.016" layer="25" ratio="10" rot="R90"/>
 <attribute name="VALUE" x="4.47675" y="4.841875" size="1.016" layer="27" ratio="10" rot="R270"/>

Commit message: Silk Screen Update
Parts:
- added U$55: OPEN_SOURCE_HW, Logo:OPENHW
- J1: value M20-7862042C64KB -> M20-7862042
- moved U$54 0.40 mm to (3.89, 72.2)
Other:
- board text added: "100n"
- board text added: "10k"
- board text added: "16MHz"
- board text added: "1M"
- board text added: "1k"
- board text added: "20p"
- board text added: "220R"
- board text added: "2x 100n"
- board text added: "2x100n"
- board text added: "2x22p"
- board text added: "330R"
- board text added: "4148"
- board text added: "ATmega 328P"
- board text added: "BC846"
- board text added: "LED+"
- board text added: "M20-7862042"
- board text added: "http://github.com/svenpetersen1965"
- board text removed: "RESIO"
Changed lines of the file:
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@@
 <layer number="14" name="Route14" color="22" fill="1" visible="no" active="no"/>
 <layer number="15" name="Route15" color="23" fill="1" visible="no" active="no"/>
-<layer number="16" name="Bottom" color="1" fill="1" visible="yes" active="yes"/>
-<layer number="17" name="Pads" color="2" fill="1" visible="yes" active="yes"/>
-<layer number="18" name="Vias" color="2" fill="1" visible="yes" active="yes"/>
+<layer number="16" name="Bottom" color="1" fill="1" visible="no" active="yes"/>
+<layer number="17" name="Pads" color="2" fill="1" visible="no" active="yes"/>
+<layer number="18" name="Vias" color="2" fill="1" visible="no" active="yes"/>
 <layer number="19" name="Unrouted" color="6" fill="1" visible="yes" active="yes"/>
 <layer number="20" name="Dimension" color="24" fill="1" visible="yes" active="yes"/>
-<layer number="21" name="tPlace" color="7" fill="1" visible="no" active="yes"/>
+<layer number="21" name="tPlace" color="7" fill="1" visible="yes" active="yes"/>
 <layer number="22" name="bPlace" color="7" fill="1" visible="no" active="yes"/>
 <layer number="23" name="tOrigins" color="15" fill="1" visible="no" active="yes"/>
 <layer number="24" name="bOrigins" color="15" fill="1" visible="no" active="yes"/>
-<layer number="25" name="tNames" color="7" fill="1" visible="no" active="yes"/>
+<layer number="25" name="tNames" color="7" fill="1" visible="yes" active="yes"/>
 <layer number="26" name="bNames" color="7" fill="1" visible="no" active="yes"/>
-<layer number="27" name="tValues" color="7" fill="1" visible="no" active="yes"/>
+<layer number="27" name="tValues" color="62" fill="1" visible="no" active="yes"/>
 <layer number="28" name="bValues" color="7" fill="1" visible="no" active="yes"/>
 <layer number="29" name="tStop" color="7" fill="3" visible="no" active="yes"/>
@@
 <layer number="45" name="Holes" color="7" fill="1" visible="no" active="yes"/>
 <layer number="46" name="Milling" color="3" fill="1" visible="no" active="yes"/>
-<layer number="47" name="Measures" color="7" fill="1" visible="no" active="yes"/>
+<layer number="47" name="Measures" color="7" fill="1" visible="yes" active="yes"/>
 <layer number="48" name="Document" color="7" fill="1" visible="yes" active="yes"/>
 <layer number="49" name="Reference" color="7" fill="1" visible="no" active="yes"/>
 <layer number="50" name="dxf" color="7" fill="1" visible="no" active="no"/>
-<layer number="51" name="tDocu" color="7" fill="1" visible="no" active="yes"/>
+<layer number="51" name="tDocu" color="7" fill="1" visible="yes" active="yes"/>
 <layer number="52" name="bDocu" color="7" fill="1" visible="no" active="yes"/>
 <layer number="53" name="tGND_GNDA" color="7" fill="1" visible="no" active="no"/>
@@
 <layer number="250" name="Descript" color="7" fill="1" visible="no" active="no"/>
 <layer number="251" name="SMDround" color="7" fill="1" visible="no" active="no"/>
+<layer number="252" name="BR-BS" color="7" fill="1" visible="no" active="yes"/>
+<layer number="253" name="BR-LS" color="7" fill="1" visible="no" active="yes"/>
 <layer number="254" name="OrgLBR" color="7" fill="1" visible="no" active="no"/>
 <layer number="255" name="routoute" color="7" fill="1" visible="yes" active="yes"/>
@@
 <text x="1.27" y="83.96375" size="1.016" layer="21" ratio="12" rot="R90">GND</text>
 <text x="15.71625" y="93.885625" size="1.016" layer="21" font="vector" align="center-right">!EXROM</text>
-<text x="15.71625" y="95.949375" size="1.016" layer="21" font="vector" align="center-right">RESIO</text>
+<text x="15.71625" y="95.949375" size="1.016" layer="21" font="vector" align="center-right">LED+</text>
 <text x="15.86" y="90.17" size="1.016" layer="21" font="vector" align="center-right">!RESET</text>
 <text x="15.875" y="88.25" size="1.27" layer="21" font="vector" align="center-right">A15</text>
@@
 <text x="51.91125" y="112.950625" size="1.778" layer="48" font="vector">2</text>
 <text x="45.72" y="106.600625" size="1.778" layer="48" font="vector">1</text>
-<text x="7.46125" y="39.21125" size="1.27" layer="21" rot="R90">C64 Keyboard Controlled
+<text x="7.540625" y="38.4175" size="1.6764" layer="21" rot="R90">C64 Keyboard Controlled
 Kernal Switch Rev. 1</text>
 <text x="19.05" y="81.5975" size="1.27" layer="16" ratio="12" rot="MR270">128/01</text>
@@
 <wire x1="8.810625" y1="100.885625" x2="8.810625" y2="99.21875" width="0.1524" layer="27"/>
 <wire x1="8.810625" y1="99.21875" x2="9.2075" y2="99.21875" width="0.1524" layer="27"/>
+<text x="18.970625" y="40.878125" size="1.016" layer="21" font="vector" rot="R90">http://github.com/svenpetersen1965</text>
+<text x="5.159375" y="78.343125" size="1.016" layer="21">330R</text>
+<text x="5.3975" y="63.5" size="1.016" layer="21">220R</text>
+<text x="10.31875" y="83.5025" size="1.016" layer="21" rot="R90">10k</text>
+<text x="7.699375" y="84.93125" size="1.016" layer="21" rot="R90">1k</text>
+<text x="5.476875" y="84.1375" size="1.016" layer="21" rot="R90">10k</text>
+<text x="5.476875" y="98.980625" size="1.016" layer="21">4148</text>
+<text x="11.985625" y="86.756875" size="1.016" layer="21" rot="R90">BC846</text>
+<text x="11.985625" y="95.5675" size="1.016" layer="21" rot="R90">10k</text>
+<text x="3.81" y="97.551875" size="1.016" layer="21" rot="R90">100n</text>
+<text x="8.016875" y="93.106875" size="1.016" layer="21">1k</text>
+<text x="8.89" y="21.74875" size="1.016" layer="21">ATmega
+328P</text>
+<text x="1.11125" y="26.19375" size="1.016" layer="21">2x100n</text>
+<text x="2.54" y="14.2875" size="1.016" layer="21" rot="R90">16MHz</text>
+<text x="5.000625" y="14.76375" size="1.016" layer="21" rot="R90">20p</text>
+<text x="8.016875" y="16.35125" size="1.016" layer="21">1M</text>
+<text x="5.87375" y="8.5725" size="1.016" layer="21">2x22p</text>
+<text x="6.429375" y="3.889375" size="1.016" layer="21">10k</text>
+<text x="16.271875" y="26.749375" size="1.016" layer="21">2x
+100n</text>
+<text x="17.78" y="40.878125" size="1.016" layer="21" rot="R90">M20-7862042</text>
 </plain>
 <attributes>
@@
 </element>
 <element name="C7" library="SMD" package="0805" value="100n" x="6.19125" y="95.87" smashed="yes" rot="R180">
-<attribute name="NAME" x="3.000375" y="98.584625" size="1.016" layer="25" ratio="10" rot="R180"/>
+<attribute name="NAME" x="1.269125" y="98.96475" size="1.016" layer="25" ratio="10" rot="R270"/>
 <attribute name="VALUE" x="7.77875" y="96.3145" size="1.016" layer="27" ratio="10" rot="R180"/>
 </element>
 <element name="CP1" library="Cutpad" package="CP_OP" value="" x="6.746875" y="6.096875" smashed="yes">
-<attribute name="NAME" x="5.810375" y="7.350875" size="1.27" layer="25"/>
+<attribute name="NAME" x="5.810375" y="7.350875" size="1.016" layer="25"/>
 </element>
 <element name="D1" library="Dioden" package="SOD80C" value="LL4148" x="6.603125" y="98.028125" smashed="yes" rot="R180">
-<attribute name="NAME" x="5.957175" y="99.21875" size="1.27" layer="25" ratio="10"/>
+<attribute name="NAME" x="5.476875" y="99.06405" size="1.27" layer="25" ratio="10" rot="R90"/>
 <attribute name="VALUE" x="4.21005" y="94.698425" size="1.27" layer="27" ratio="10" rot="R90"/>
 </element>
@@
 <attribute name="PACKAGE" value="TQFP-32" x="37.24125" y="14.91375" size="1.778" layer="27" display="off"/>
 <attribute name="SUPPLIER" value="ATMEL" x="37.24125" y="14.91375" size="1.778" layer="27" display="off"/>
-<attribute name="VALUE" x="3.72085" y="27.807225" size="1.27" layer="27" ratio="10" rot="SR0"/>
-</element>
-<element name="J1" library="HARWIN" package="C64_KEYBOARD" value="M20-7862042C64KB" x="14" y="57.13" smashed="yes" rot="R90">
+<attribute name="VALUE" x="19.1034" y="28.0096" size="1.016" layer="27" ratio="10" rot="SR90"/>
+</element>
+<element name="J1" library="HARWIN" package="C64_KEYBOARD" value="M20-7862042" x="14" y="57.13" smashed="yes" rot="R90">
 <attribute name="NAME" x="13.23125" y="30.1325" size="1.27" layer="25"/>
 <attribute name="SPICEPREFIX" value="X" x="43.21" y="96.5" size="1.778" layer="27" rot="R90" display="off"/>
@@
 </element>
 <element name="R1" library="SMD" package="0805" value="10k" x="10.00125" y="97.060625" smashed="yes" rot="R90">
-<attribute name="NAME" x="12.17525" y="97.488375" size="1.016" layer="25" ratio="10" rot="R90"/>
+<attribute name="NAME" x="11.049" y="97.99725" size="1.016" layer="25" ratio="10"/>
 <attribute name="VALUE" x="10.44575" y="95.473125" size="1.016" layer="27" ratio="10" rot="R90"/>
 </element>
@@
 </element>
 <element name="R3" library="SMD" package="0805" value="1M" x="7.77875" y="15.38375" smashed="yes" rot="R180">
-<attribute name="NAME" x="8.001" y="17.54275" size="1.016" layer="25" ratio="10" rot="R180"/>
+<attribute name="NAME" x="5.969" y="16.42975" size="1.016" layer="25" ratio="10"/>
 <attribute name="VALUE" x="9.36625" y="15.82825" size="1.016" layer="27" ratio="10" rot="R180"/>
 </element>
@@
 </element>
 <element name="R7" library="SMD" package="0805" value="1k" x="6.19125" y="93.33" smashed="yes">
-<attribute name="NAME" x="8.98525" y="93.2665" size="1.016" layer="25" ratio="10" rot="R90"/>
+<attribute name="NAME" x="8.1765" y="94.0435" size="1.016" layer="25" ratio="10"/>
 <attribute name="VALUE" x="4.60375" y="92.8855" size="1.016" layer="27" ratio="10"/>
 </element>
@@
 <attribute name="VALUE" x="4.47675" y="4.841875" size="1.016" layer="27" ratio="10" rot="R270"/>
 </element>
-<element name="U$54" library="Logo" package="SVEN_TAG" value="" x="4.1275" y="71.91375" smashed="yes"/>
+<element name="U$54" library="Logo" package="SVEN_TAG" value="" x="3.889375" y="72.23125" smashed="yes"/>
+<element name="U$55" library="Logo" package="OPENHW" value="OPEN_SOURCE_HW" x="8.651875" y="27.14625" smashed="yes" rot="R90"/>
 </elements>
 <signals>
