File: Rev. 1/Eagle/C64_Kernal_Switch.sch (EAGLE design)
At the start: 27 parts, among them IC1 ATMEGA328P-AU, J1 M20-7862042C64KB, J2 WSL 6G, J3 n/a, Q1 BC846, X1 FOXSLF/160-20

Commit message: Rev. 1 Documentation released
The final documentation is released
Parts:
- R10: value 1k -> n/a
- R9: value 220R -> 330R
Changed lines of the file:
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@@
 <?xml version="1.0" encoding="utf-8"?>
 <!DOCTYPE eagle SYSTEM "eagle.dtd">
-<eagle version="9.2.2">
+<eagle version="9.5.2">
 <drawing>
 <settings>
@@
 <part name="R8" library="SMD" deviceset="R-0805" device="" value="220R"/>
 <part name="U$40" library="!GRAFIK" deviceset="OUT" device=""/>
-<part name="R9" library="SMD" deviceset="R-0805" device="" value="220R"/>
-<part name="R10" library="SMD" deviceset="R-0805" device="" value="1k"/>
+<part name="R9" library="SMD" deviceset="R-0805" device="" value="330R"/>
+<part name="R10" library="SMD" deviceset="R-0805" device="" value="n/a"/>
 <part name="U$53" library="!pownet" deviceset="GND" device=""/>
 </parts>

Commit message: Silk Screen Update
Parts:
- added U$55: OPEN_SOURCE_HW, Logo:OPEN_SOURCE_HW
- J1: value M20-7862042C64KB -> M20-7862042
Other:
- note added: "https://github.com/svenpetersen1965"
Changed lines of the file:
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@@
 <layer number="250" name="Descript" color="7" fill="1" visible="no" active="no"/>
 <layer number="251" name="SMDround" color="7" fill="1" visible="no" active="no"/>
+<layer number="252" name="BR-BS" color="7" fill="1" visible="no" active="yes"/>
+<layer number="253" name="BR-LS" color="7" fill="1" visible="no" active="yes"/>
 <layer number="254" name="OrgLBR" color="7" fill="1" visible="no" active="no"/>
 <layer number="255" name="routoute" color="7" fill="1" visible="yes" active="yes"/>
@@
 <parts>
 <part name="U$1" library="DOC_IBSP" deviceset="A3/" device=""/>
-<part name="J1" library="HARWIN" deviceset="M20-7862042" device="C64KB" value="M20-7862042C64KB">
+<part name="J1" library="HARWIN" deviceset="M20-7862042" device="C64KB" value="M20-7862042">
 <attribute name="SPICEPREFIX" value="X"/>
 </part>
@@
 <part name="R10" library="SMD" deviceset="R-0805" device="" value="n/a"/>
 <part name="U$53" library="!pownet" deviceset="GND" device=""/>
+<part name="U$55" library="Logo" deviceset="OPEN_SOURCE_HW" device=""/>
 </parts>
 <sheets>
@@
 <wire x1="67.31" y1="210.82" x2="67.31" y2="209.55" width="0.1524" layer="96"/>
 <wire x1="67.31" y1="209.55" x2="64.77" y2="209.55" width="0.1524" layer="96"/>
+<text x="279.4" y="7.62" size="2.54" layer="95">https://github.com/svenpetersen1965</text>
 </plain>
 <instances>
@@
 <attribute name="VALUE" x="279.7175" y="163.195" size="1.524" layer="96"/>
 </instance>
+<instance part="U$55" gate="G$1" x="238.76" y="7.62" smashed="yes"/>
 </instances>
 <busses>
